File: hardware/hhv-dcdarknet.brd (EAGLE design)
At the start: 43.2 x 75.8 mm, 61 parts, among them IC1 ATMEGA328P-PU, U1 RCV, U2 VT1045CTO262-H, X2 USB

Commit message: Update hhv-dcdarknet.brd
Updated version for DC23.  Adjustments on layout and increased pad sizes and spacing.  Silk screen has not been updated yet.
Parts:
- JP10, JP11, JP12, JP13, JP14, JP15, JP16, JP17, JP18, JP19, JP20, JP21, JP22, JP23, JP24, JP25, JP26, JP27, JP28, JP29, JP3, JP30, JP4, JP5, JP6, JP7, JP8, JP9: device adafruit:1X1-SMALL -> adafruit:1X1-SMALL_CUT
- R10, R7, R8, R9: device SparkFun:0805 -> SparkFun:1206
- R6: value 2.2K -> 1.5K
- moved R8 0.95 mm to (75.9, 66.7)
- moved R9 0.95 mm to (54.0, 66.7)
Routing:
- net PIN5: track 8.65 -> 7.72 mm
- net PIN18: track 75.1 -> 75.7 mm
- added copper zone on layer 1, net N$10
- added copper zone on layer 1, net N$9
