File: hardware/hhv-dcdarknet.sch (EAGLE design)
At the start: 61 parts, among them IC1 ATMEGA328P-PU, SW1 SWITCH_TACTILETACTILE-2PIN, U1 RCV, U2 VT1045CTO262-H, X2 USB

Commit message: Update hhv-dcdarknet.sch
Updated board for DC23.
Parts:
- JP10, JP11, JP12, JP13, JP14, JP15, JP16, JP17, JP18, JP19, JP20, JP21, JP22, JP23, JP24, JP25, JP26, JP27, JP28, JP29, JP3, JP30, JP4, JP5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: device adafruit:PINHD-1X11X1-SMALL -> adafruit:PINHD-1X11X1_SQUARE
- R10, R7, R8, R9: device SparkFun:RESISTOR0805-RES -> SparkFun:RESISTOR1206
- R6: value 2.2K -> 1.5K
