File: hardware/hhv-dcdarknet-varient-2.sch (EAGLE design)
At the start: 62 parts, among them IC1 ATMEGA328P-PU, SW1 SWITCH_TACTILETACTILE-2PIN, U1 RCV, U2 VT1045CTO262-H, X2 USB

Commit message: Updated Eagle files for the 2015 boards.
Parts:
- JP24, JP25, JP27, JP29: device adafruit:PINHD-1X11X1-SMALL -> adafruit:PINHD-1X11X1_SQUARE
- JP28: device adafruit:PINHD-1X11X1_SQUARE -> adafruit:PINHD-1X11X1-SMALL
Changed lines of the file:
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@@
 <part name="JP22" library="adafruit" deviceset="PINHD-1X1" device="1X1_SQUARE"/>
 <part name="JP23" library="adafruit" deviceset="PINHD-1X1" device="1X1_SQUARE"/>
-<part name="JP24" library="adafruit" deviceset="PINHD-1X1" device="1X1-SMALL"/>
-<part name="JP25" library="adafruit" deviceset="PINHD-1X1" device="1X1-SMALL"/>
+<part name="JP24" library="adafruit" deviceset="PINHD-1X1" device="1X1_SQUARE"/>
+<part name="JP25" library="adafruit" deviceset="PINHD-1X1" device="1X1_SQUARE"/>
 <part name="JP26" library="adafruit" deviceset="PINHD-1X1" device="1X1_SQUARE"/>
-<part name="JP27" library="adafruit" deviceset="PINHD-1X1" device="1X1-SMALL"/>
-<part name="JP28" library="adafruit" deviceset="PINHD-1X1" device="1X1_SQUARE"/>
-<part name="JP29" library="adafruit" deviceset="PINHD-1X1" device="1X1-SMALL"/>
+<part name="JP27" library="adafruit" deviceset="PINHD-1X1" device="1X1_SQUARE"/>
+<part name="JP28" library="adafruit" deviceset="PINHD-1X1" device="1X1-SMALL"/>
+<part name="JP29" library="adafruit" deviceset="PINHD-1X1" device="1X1_SQUARE"/>
 <part name="JP30" library="adafruit" deviceset="PINHD-1X1" device="1X1-SMALL"/>
 <part name="C3" library="adafruit" deviceset="C-US" device="025-030X050" value=".1uf"/>
