File: hardware/hhv-dcdarknet-varient-4.brd (EAGLE design)
At the start: 43.2 x 75.8 mm, 62 parts, among them IC1 ATMEGA328P-PU, U1 RCV, U2 VT1045CTO262-H, X2 USB

Commit message: Updated Eagle files for the 2015 boards.
Parts:
- JP24, JP25, JP27, JP29: device adafruit:1X1-SMALL -> adafruit:1X1-SMALL_CUT
- JP26: device adafruit:1X1-SMALL_CUT -> adafruit:1X1-SMALL
Other:
- board text added: "36390 45539 12903 15061"
- board text added: "39754 35656 64833 94926"
- board text added: "59648 34191"
- board text added: "61470 80274 49444 87883"
- board text removed: "17185 65867 58278 18586"
- board text removed: "48269 27789"
- board text removed: "69667 18282 71718 71667"
- board text removed: "86697 06566 65707 70677"
Changed lines of the file:
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@@
 <wire x1="56.515" y1="61.2775" x2="56.67375" y2="61.356875" width="0.6096" layer="41"/>
 <text x="46.99" y="52.3875" size="0.8128" layer="121" rot="R90">USB Tx</text>
-<text x="77.33665" y="8.226425" size="1.27" layer="122" font="vector" distance="45" rot="MR0">69667
-18282
-71718
-71667</text>
+<text x="77.33665" y="8.226425" size="1.27" layer="122" font="vector" distance="45" rot="MR0">61470
+80274
+49444
+87883</text>
 <wire x1="76.04125" y1="21.43125" x2="75.08875" y2="21.43125" width="0.254" layer="122"/>
 <wire x1="75.08875" y1="21.43125" x2="74.13625" y2="21.43125" width="0.254" layer="122"/>
@@
 <vertex x="62.865" y="52.3875"/>
 </polygon>
-<text x="70.8279" y="8.226425" size="1.27" layer="122" font="vector" distance="45" rot="MR0">17185
-65867
-58278
-18586</text>
-<text x="64.31915" y="8.226425" size="1.27" layer="122" font="vector" distance="45" rot="MR0">86697
-06566
-65707
-70677</text>
-<text x="57.8104" y="8.226425" size="1.27" layer="122" font="vector" distance="45" rot="MR0">48269
-27789</text>
+<text x="70.8279" y="8.226425" size="1.27" layer="122" font="vector" distance="45" rot="MR0">36390
+45539
+12903
+15061</text>
+<text x="64.31915" y="8.226425" size="1.27" layer="122" font="vector" distance="45" rot="MR0">39754
+35656
+64833
+94926</text>
+<text x="57.8104" y="8.226425" size="1.27" layer="122" font="vector" distance="45" rot="MR0">59648
+34191</text>
 </plain>
 <attributes>
@@
 <element name="JP22" library="adafruit" package="1X1-SMALL_CUT" value="" x="48.26" y="36.83"/>
 <element name="JP23" library="adafruit" package="1X1-SMALL_CUT" value="" x="48.26" y="34.29"/>
-<element name="JP24" library="adafruit" package="1X1-SMALL" value="" x="48.26" y="31.75"/>
-<element name="JP25" library="adafruit" package="1X1-SMALL" value="" x="48.26" y="29.21"/>
-<element name="JP26" library="adafruit" package="1X1-SMALL_CUT" value="" x="48.26" y="26.67"/>
-<element name="JP27" library="adafruit" package="1X1-SMALL" value="" x="48.26" y="24.13"/>
+<element name="JP24" library="adafruit" package="1X1-SMALL_CUT" value="" x="48.26" y="31.75"/>
+<element name="JP25" library="adafruit" package="1X1-SMALL_CUT" value="" x="48.26" y="29.21"/>
+<element name="JP26" library="adafruit" package="1X1-SMALL" value="" x="48.26" y="26.67"/>
+<element name="JP27" library="adafruit" package="1X1-SMALL_CUT" value="" x="48.26" y="24.13"/>
 <element name="JP28" library="adafruit" package="1X1-SMALL_CUT" value="" x="48.26" y="21.59"/>
-<element name="JP29" library="adafruit" package="1X1-SMALL" value="" x="48.26" y="19.05"/>
+<element name="JP29" library="adafruit" package="1X1-SMALL_CUT" value="" x="48.26" y="19.05"/>
 <element name="JP30" library="adafruit" package="1X1-SMALL" value="" x="48.26" y="16.51"/>
 <element name="C3" library="adafruit" package="C025-030X050" value=".1uf" x="75.40625" y="17.93875" smashed="yes" rot="R270">
@@
 </element>
 <element name="LED4" library="SparkFun" package="LED-1206" value="" x="74.45375" y="62.38875" smashed="yes" rot="MR180">
-<attribute name="NAME" x="71.8185" y="64.48425" size="0.8128" layer="26" rot="MR180"/>
+<attribute name="NAME" x="71.65975" y="64.48425" size="0.8128" layer="26" rot="MR180"/>
 <attribute name="VALUE" x="73.43775" y="64.16675" size="0.4064" layer="28" rot="MR180"/>
 </element>
 <element name="LED5" library="SparkFun" package="LED-1206" value="" x="55.08625" y="62.38875" smashed="yes" rot="MR180">
-<attribute name="NAME" x="55.032275" y="64.468375" size="0.8128" layer="26" rot="MR180"/>
+<attribute name="NAME" x="55.191025" y="64.468375" size="0.8128" layer="26" rot="MR180"/>
 <attribute name="VALUE" x="54.07025" y="64.16675" size="0.4064" layer="28" rot="MR180"/>
 </element>
@@
 </element>
 <element name="R7" library="SparkFun" package="1206" value="" x="83.185" y="63.8175" smashed="yes" rot="MR270">
-<attribute name="NAME" x="83.78825" y="66.548" size="0.8128" layer="26" rot="MR0"/>
+<attribute name="NAME" x="83.78825" y="66.38925" size="0.8128" layer="26" rot="MR0"/>
 <attribute name="VALUE" x="84.582" y="64.8335" size="0.4064" layer="28" rot="MR270"/>
 </element>
 <element name="R8" library="SparkFun" package="1206" value="" x="75.8825" y="66.675" smashed="yes" rot="MR270">
-<attribute name="NAME" x="74.58075" y="66.38925" size="0.8128" layer="26" rot="MR0"/>
+<attribute name="NAME" x="74.7395" y="66.2305" size="0.8128" layer="26" rot="MR0"/>
 <attribute name="VALUE" x="77.2795" y="67.691" size="0.4064" layer="28" rot="MR270"/>
 </element>
