File: hardware/hhv-dcdarknet-varient-6.brd (EAGLE design)
At the start: 43.2 x 75.8 mm, 62 parts, among them IC1 ATMEGA328P-PU, U1 RCV, U2 VT1045CTO262-H, X2 USB

Commit message: Updated Eagle files for the 2015 boards.
Parts:
- JP25, JP29: device adafruit:1X1-SMALL -> adafruit:1X1-SMALL_CUT
Other:
- board text added: "76383 54112 38126 37950"
- board text added: "79364 89734 46175 65047"
- board text added: "82309 65870"
- board text added: "97857 90276 02679 53162"
- board text removed: "17185 65867 58278 18586"
- board text removed: "48269 27789"
- board text removed: "69667 18282 71718 71667"
- board text removed: "86697 06566 65707 70677"
Changed lines of the file:
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@@
 <wire x1="56.515" y1="61.2775" x2="56.67375" y2="61.356875" width="0.6096" layer="41"/>
 <text x="46.99" y="52.3875" size="0.8128" layer="121" rot="R90">USB Tx</text>
-<text x="77.33665" y="8.226425" size="1.27" layer="122" font="vector" distance="45" rot="MR0">69667
-18282
-71718
-71667</text>
+<text x="77.33665" y="8.226425" size="1.27" layer="122" font="vector" distance="45" rot="MR0">79364
+89734
+46175
+65047</text>
 <wire x1="76.04125" y1="21.43125" x2="75.08875" y2="21.43125" width="0.254" layer="122"/>
 <wire x1="75.08875" y1="21.43125" x2="74.13625" y2="21.43125" width="0.254" layer="122"/>
@@
 <vertex x="62.865" y="52.3875"/>
 </polygon>
-<text x="70.8279" y="8.226425" size="1.27" layer="122" font="vector" distance="45" rot="MR0">17185
-65867
-58278
-18586</text>
-<text x="64.31915" y="8.226425" size="1.27" layer="122" font="vector" distance="45" rot="MR0">86697
-06566
-65707
-70677</text>
-<text x="57.8104" y="8.226425" size="1.27" layer="122" font="vector" distance="45" rot="MR0">48269
-27789</text>
+<text x="70.8279" y="8.226425" size="1.27" layer="122" font="vector" distance="45" rot="MR0">97857
+90276
+02679
+53162</text>
+<text x="64.31915" y="8.226425" size="1.27" layer="122" font="vector" distance="45" rot="MR0">76383
+54112
+38126
+37950</text>
+<text x="57.8104" y="8.226425" size="1.27" layer="122" font="vector" distance="45" rot="MR0">82309
+65870</text>
 </plain>
 <attributes>
@@
 <element name="JP23" library="adafruit" package="1X1-SMALL_CUT" value="" x="48.26" y="34.29"/>
 <element name="JP24" library="adafruit" package="1X1-SMALL" value="" x="48.26" y="31.75"/>
-<element name="JP25" library="adafruit" package="1X1-SMALL" value="" x="48.26" y="29.21"/>
+<element name="JP25" library="adafruit" package="1X1-SMALL_CUT" value="" x="48.26" y="29.21"/>
 <element name="JP26" library="adafruit" package="1X1-SMALL_CUT" value="" x="48.26" y="26.67"/>
 <element name="JP27" library="adafruit" package="1X1-SMALL" value="" x="48.26" y="24.13"/>
 <element name="JP28" library="adafruit" package="1X1-SMALL_CUT" value="" x="48.26" y="21.59"/>
-<element name="JP29" library="adafruit" package="1X1-SMALL" value="" x="48.26" y="19.05"/>
+<element name="JP29" library="adafruit" package="1X1-SMALL_CUT" value="" x="48.26" y="19.05"/>
 <element name="JP30" library="adafruit" package="1X1-SMALL" value="" x="48.26" y="16.51"/>
 <element name="C3" library="adafruit" package="C025-030X050" value=".1uf" x="75.40625" y="17.93875" smashed="yes" rot="R270">
